File: der_switch_new.kicad_pcb (KiCad board)
At the start: 2 copper layers, 74 parts, among them J1 JK0654219, J2 JK0654219, J3 JK0654219, J4 JK0654219, J5 JK0654219, U1 KSZ9477S

Commit message: update pin naming. use _P/_N to allow optiomisation for differential signal
Signed-off-by: Oleksij Rempel <linux@rempel-privat.de>
Parts:
- moved R2 118.5 mm to (204.0, 132.5)
- moved C42 109.9 mm to (205.6, 125.8), turned to 180 degrees
- moved C41 100.0 mm to (206.1, 122.5), turned to 180 degrees
- moved U1 43.9 mm to (183.5, 91.5)
- moved J4 28.3 mm to (238.6, 55.0)
- moved J3 24.3 mm to (238.6, 75.0)
- moved J2 19.0 mm to (238.6, 95.0)
- moved J1 12.1 mm to (238.6, 115.0)
- moved R3 10.9 mm to (140.8, 44.4)
- moved J5 8.43 mm to (238.6, 135.0)
Routing:
- net Earth: track 0.00 -> 96.1 mm
- added copper zone on In3.Cu, net GND
Other:
- copper layers 2 -> 6
Changed lines of the file:
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@@
   (layers
     (0 "F.Cu" signal)
+    (1 "In1.Cu" signal)
+    (2 "In2.Cu" signal)
+    (3 "In3.Cu" signal)
+    (4 "In4.Cu" signal)
     (31 "B.Cu" signal)
     (32 "B.Adhes" user "B.Adhesive")
@@
     (48 "B.Fab" user)
     (49 "F.Fab" user)
-    (50 "User.1" user)
-    (51 "User.2" user)
-    (52 "User.3" user)
-    (53 "User.4" user)
-    (54 "User.5" user)
-    (55 "User.6" user)
-    (56 "User.7" user)
-    (57 "User.8" user)
-    (58 "User.9" user)
   )
   (setup
+    (stackup
+      (layer "F.SilkS" (type "Top Silk Screen"))
+      (layer "F.Paste" (type "Top Solder Paste"))
+      (layer "F.Mask" (type "Top Solder Mask") (color "Green") (thickness 0.01))
+      (layer "F.Cu" (type "copper") (thickness 0.035))
+      (layer "dielectric 1" (type "core") (thickness 0.274) (material "FR4") (epsilon_r 4.5) (loss_tangent 0.02))
+      (layer "In1.Cu" (type "copper") (thickness 0.035))
+      (layer "dielectric 2" (type "prepreg") (thickness 0.274) (material "FR4") (epsilon_r 4.5) (loss_tangent 0.02))
+      (layer "In2.Cu" (type "copper") (thickness 0.035))
+      (layer "dielectric 3" (type "core") (thickness 0.274) (material "FR4") (epsilon_r 4.5) (loss_tangent 0.02))
+      (layer "In3.Cu" (type "copper") (thickness 0.035))
+      (layer "dielectric 4" (type "prepreg") (thickness 0.274) (material "FR4") (epsilon_r 4.5) (loss_tangent 0.02))
+      (layer "In4.Cu" (type "copper") (thickness 0.035))
+      (layer "dielectric 5" (type "core") (thickness 0.274) (material "FR4") (epsilon_r 4.5) (loss_tangent 0.02))
+      (layer "B.Cu" (type "copper") (thickness 0.035))
+      (layer "B.Mask" (type "Bottom Solder Mask") (color "Green") (thickness 0.01))
+      (layer "B.Paste" (type "Bottom Solder Paste"))
+      (layer "B.SilkS" (type "Bottom Silk Screen"))
+      (copper_finish "None")
+      (dielectric_constraints no)
+    )
     (pcbplotparams
       (layerselection 0x00010fc_ffffffff)
@@
   )
   (footprint "Connector_RJ:RJ45_Pulse_JK0654219NL_Horizontal" (layer "F.Cu")
-    (at 241.3 50.8)
+    (at 238.585 74.9845)
     (descr "10/100/1000 Base-T RJ45 single port with LEDs https://media.digikey.com/pdf/Data%20Sheets/Pulse%20PDFs/JK%20Series.pdf#page=2")
     (tags "RJ45 8p8c ethernet")
@@
   )
   (footprint "footprints:TQFP-128_14x14mm_P0.4mm_EP10x10mm_ThermalVias" (layer "F.Cu")
-    (at 139.7 88.9 180)
+    (at 183.5 91.5 180)
     (descr "TQFP128 14x14 / TQFP128 CASE 932BB (see ON Semiconductor 932BB.PDF)")
     (tags "QFP 0.4")
@@
   )
   (footprint "Connector_RJ:RJ45_Pulse_JK0654219NL_Horizontal" (layer "F.Cu")
-    (at 241.3 127)
+    (at 238.585 134.9845)
     (descr "10/100/1000 Base-T RJ45 single port with LEDs https://media.digikey.com/pdf/Data%20Sheets/Pulse%20PDFs/JK%20Series.pdf#page=2")
     (tags "RJ45 8p8c ethernet")
@@
   )
   (footprint "Connector_RJ:RJ45_Pulse_JK0654219NL_Horizontal" (layer "F.Cu")
-    (at 241.3 76.2)
+    (at 238.585 94.9845)
     (descr "10/100/1000 Base-T RJ45 single port with LEDs https://media.digikey.com/pdf/Data%20Sheets/Pulse%20PDFs/JK%20Series.pdf#page=2")
     (tags "RJ45 8p8c ethernet")
@@
   )
   (footprint "Connector_RJ:RJ45_Pulse_JK0654219NL_Horizontal" (layer "F.Cu")
-    (at 238.76 102.87)
+    (at 238.585 114.9845)
     (descr "10/100/1000 Base-T RJ45 single port with LEDs https://media.digikey.com/pdf/Data%20Sheets/Pulse%20PDFs/JK%20Series.pdf#page=2")
     (tags "RJ45 8p8c ethernet")
@@
   )
   (footprint "Connector_RJ:RJ45_Pulse_JK0654219NL_Horizontal" (layer "F.Cu")
-    (at 238.76 26.67)
+    (at 238.585 54.9845)
     (descr "10/100/1000 Base-T RJ45 single port with LEDs https://media.digikey.com/pdf/Data%20Sheets/Pulse%20PDFs/JK%20Series.pdf#page=2")
     (tags "RJ45 8p8c ethernet")
@@
   )
   (footprint "Resistor_SMD:R_0805_2012Metric_Pad1.20x1.40mm_HandSolder" (layer "F.Cu")
-    (at 183.49 15.82)
+    (at 204 132.5)
     (descr "Resistor SMD 0805 (2012 Metric), square (rectangular) end terminal, IPC_7351 nominal with elongated pad for handsoldering. (Body size source: IPC-SM-782 page 72, https://www.pcb-3d.com/wordpress/wp-content/uploads/ipc-sm-782a_amendment_1_and_2.pdf), generated with kicad-footprint-generator")
     (tags "resistor handsolder")
@@
   )
   (footprint "Capacitor_SMD:C_0402_1005Metric_Pad0.74x0.62mm_HandSolder" (layer "F.Cu")
-    (at 155.61 36.13)
+    (at 206.0675 122.5 180)
     (descr "Capacitor SMD 0402 (1005 Metric), square (rectangular) end terminal, IPC_7351 nominal with elongated pad for handsoldering. (Body size source: IPC-SM-782 page 76, https://www.pcb-3d.com/wordpress/wp-content/uploads/ipc-sm-782a_amendment_1_and_2.pdf), generated with kicad-footprint-generator")
     (tags "capacitor handsolder")
@@
     (fp_line (start 0.5 0.25) (end -0.5 0.25) (layer "F.Fab") (width 0.1))
     (fp_line (start -0.5 0.25) (end -0.5 -0.25) (layer "F.Fab") (width 0.1))
-    (pad "1" smd roundrect (at -0.5675 0) (locked) (size 0.735 0.62) (layers "F.Cu" "F.Paste" "F.Mask") (roundrect_rratio 0.25)
+    (pad "1" smd roundrect (at -0.5675 0 180) (locked) (size 0.735 0.62) (layers "F.Cu" "F.Paste" "F.Mask") (roundrect_rratio 0.25)
       (net 10 "Net-(C41-Pad1)"))
-    (pad "2" smd roundrect (at 0.5675 0) (locked) (size 0.735 0.62) (layers "F.Cu" "F.Paste" "F.Mask") (roundrect_rratio 0.25)
+    (pad "2" smd roundrect (at 0.5675 0 180) (locked) (size 0.735 0.62) (layers "F.Cu" "F.Paste" "F.Mask") (roundrect_rratio 0.25)
       (net 1 "GND"))
     (model "${KICAD6_3DMODEL_DIR}/Capacitor_SMD.3dshapes/C_0402_1005Metric.wrl"
@@
   )
   (footprint "Resistor_SMD:R_0805_2012Metric_Pad1.20x1.40mm_HandSolder" (layer "F.Cu")
-    (at 148.42 36.62)
+    (at 140.825 44.375)
     (descr "Resistor SMD 0805 (2012 Metric), square (rectangular) end terminal, IPC_7351 nominal with elongated pad for handsoldering. (Body size source: IPC-SM-782 page 72, https://www.pcb-3d.com/wordpress/wp-content/uploads/ipc-sm-782a_amendment_1_and_2.pdf), generated with kicad-footprint-generator")
     (tags "resistor handsolder")
@@
   )
   (footprint "Capacitor_SMD:C_0402_1005Metric_Pad0.74x0.62mm_HandSolder" (layer "F.Cu")
-    (at 182.72 18.28)
+    (at 205.575 125.825 180)
     (descr "Capacitor SMD 0402 (1005 Metric), square (rectangular) end terminal, IPC_7351 nominal with elongated pad for handsoldering. (Body size source: IPC-SM-782 page 76, https://www.pcb-3d.com/wordpress/wp-content/uploads/ipc-sm-782a_amendment_1_and_2.pdf), generated with kicad-footprint-generator")
     (tags "capacitor handsolder")
@@
     (fp_line (start 0.5 -0.25) (end 0.5 0.25) (layer "F.Fab") (width 0.1))
     (fp_line (start 0.5 0.25) (end -0.5 0.25) (layer "F.Fab") (width 0.1))
-    (pad "1" smd roundrect (at -0.5675 0) (locked) (size 0.735 0.62) (layers "F.Cu" "F.Paste" "F.Mask") (roundrect_rratio 0.25)
+    (pad "1" smd roundrect (at -0.5675 0 180) (locked) (size 0.735 0.62) (layers "F.Cu" "F.Paste" "F.Mask") (roundrect_rratio 0.25)
       (net 11 "Net-(C42-Pad1)"))
-    (pad "2" smd roundrect (at 0.5675 0) (locked) (size 0.735 0.62) (layers "F.Cu" "F.Paste" "F.Mask") (roundrect_rratio 0.25)
+    (pad "2" smd roundrect (at 0.5675 0 180) (locked) (size 0.735 0.62) (layers "F.Cu" "F.Paste" "F.Mask") (roundrect_rratio 0.25)
       (net 1 "GND"))
     (model "${KICAD6_3DMODEL_DIR}/Capacitor_SMD.3dshapes/C_0402_1005Metric.wrl"
@@
     )
   )
+  (segment (start 257 52) (end 257 68.129) (width 0.25) (layer "B.Cu") (net 61))
+  (segment (start 257 68.129) (end 257 72) (width 0.25) (layer "B.Cu") (net 61))
+  (segment (start 257 88.129) (end 257 92) (width 0.25) (layer "B.Cu") (net 61))
+  (segment (start 257 108.129) (end 257 112) (width 0.25) (layer "B.Cu") (net 61))
+  (segment (start 257 112) (end 257 128.129) (width 0.25) (layer "B.Cu") (net 61))
+  (segment (start 257 72) (end 257 88.129) (width 0.25) (layer "B.Cu") (net 61))
+  (segment (start 257 128.129) (end 257 132) (width 0.25) (layer "B.Cu") (net 61))
+  (segment (start 257 132) (end 257 148.129) (width 0.25) (layer "B.Cu") (net 61))
+  (segment (start 257 92) (end 257 108.129) (width 0.25) (layer "B.Cu") (net 61))
+  (zone (net 1) (net_name "GND") (layer "In3.Cu") (hatch edge 0.508)
+    (connect_pads (clearance 0.508))
+    (min_thickness 0.254) (filled_areas_thickness no)
+    (fill yes (thermal_gap 0.508) (thermal_bridge_width 0.508))
+    (polygon
+      (pts
+        (xy 245 160)
+        (xy 110 160.5)
+        (xy 110 40)
+        (xy 245 40)
+      )
+    )
+  )
