File: ethernet_ports.kicad_sch (KiCad schematic)
At the start: 8 parts, among them J5 JK0654219, U1 KSZ9477S

Commit message: add TQFP-128_14x14mm_P0.4mm_EP10x10mm_ThermalVias footprint
and assign it to the ksz chip

Signed-off-by: Oleksij Rempel <linux@rempel-privat.de>
Parts:
- U1: footprint Package_QFP:TQFP-128_14x14mm_P0.4mm -> footprints:TQFP-128_14x14mm_P0.4mm_EP10x10mm_ThermalVias
Connections:
- net P1_A_M is gone; now on net P5_A_M: J5.10 (MX1-)
- net P1_A_P is gone; now on net P5_A_P: J5.11 (MX1+)
- net P1_B_M is gone; now on net P5_B_M: J5.5 (MX2-)
- net P1_B_P is gone; now on net P5_B_P: J5.4 (MX2+)
- net P1_C_M is gone; now on net P5_C_M: J5.2 (MX3-)
- net P1_C_P is gone; now on net P5_C_P: J5.3 (MX3+)
- net P1_D_M is gone; now on net P5_D_M: J5.9 (MX4-)
- net P1_D_P is gone; now on net P5_D_P: J5.8 (MX4+)
- net P1_LED0 is gone; now on net P5_LED0: J5.15 (LED1-)
- net P1_LED1 is gone; now on net P5_LED1: J5.13 (LED2-)
Changed lines of the file:
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@@
     (effects (font (size 1.27 1.27)) (justify right bottom))
   )
-  (label "P1_LED0" (at 215.9 38.1 180)
+  (label "P5_LED0" (at 215.9 38.1 180)
     (effects (font (size 1.27 1.27)) (justify right bottom))
   )
-  (label "P1_A_P" (at 215.9 43.18 180)
+  (label "P5_A_P" (at 215.9 43.18 180)
     (effects (font (size 1.27 1.27)) (justify right bottom))
   )
-  (label "P1_A_M" (at 215.9 48.26 180)
+  (label "P5_A_M" (at 215.9 48.26 180)
     (effects (font (size 1.27 1.27)) (justify right bottom))
   )
-  (label "P1_B_P" (at 215.9 53.34 180)
+  (label "P5_B_P" (at 215.9 53.34 180)
     (effects (font (size 1.27 1.27)) (justify right bottom))
   )
-  (label "P1_B_M" (at 215.9 58.42 180)
+  (label "P5_B_M" (at 215.9 58.42 180)
     (effects (font (size 1.27 1.27)) (justify right bottom))
   )
-  (label "P1_C_P" (at 215.9 63.5 180)
+  (label "P5_C_P" (at 215.9 63.5 180)
     (effects (font (size 1.27 1.27)) (justify right bottom))
   )
-  (label "P1_C_M" (at 215.9 68.58 180)
+  (label "P5_C_M" (at 215.9 68.58 180)
     (effects (font (size 1.27 1.27)) (justify right bottom))
   )
-  (label "P1_D_P" (at 215.9 73.66 180)
+  (label "P5_D_P" (at 215.9 73.66 180)
     (effects (font (size 1.27 1.27)) (justify right bottom))
   )
-  (label "P1_D_M" (at 215.9 78.74 180)
+  (label "P5_D_M" (at 215.9 78.74 180)
     (effects (font (size 1.27 1.27)) (justify right bottom))
   )
-  (label "P1_LED1" (at 215.9 86.36 180)
+  (label "P5_LED1" (at 215.9 86.36 180)
     (effects (font (size 1.27 1.27)) (justify right bottom))
   )
@@
     (property "Reference" "U1" (id 0) (at 139.7 40.64 0))
     (property "Value" "KSZ9477S" (id 1) (at 139.7 43.18 0))
-    (property "Footprint" "Package_QFP:TQFP-128_14x14mm_P0.4mm" (id 2) (at 121.666 82.042 0)
+    (property "Footprint" "footprints:TQFP-128_14x14mm_P0.4mm_EP10x10mm_ThermalVias" (id 2) (at 121.666 82.042 0)
       (effects (font (size 1.27 1.27)) hide)
     )

Commit message: update pin naming. use _P/_N to allow optiomisation for differential signal
Signed-off-by: Oleksij Rempel <linux@rempel-privat.de>
Parts:
- renumbered U1 to U
Changed lines of the file:
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@@
-(kicad_sch (version 20201015) (generator eeschema)
+(kicad_sch (version 20210126) (generator eeschema)
   (paper "A4")
   (junction (at 194.31 55.88) (diameter 0.9144) (color 0 0 0 0))
@@
       (effects (font (size 1.27 1.27)) hide)
     )
+    (pin "1")
   )
   (symbol (lib_id "power:+3V3") (at 193.04 35.56 0) (unit 1)
@@
       (effects (font (size 1.27 1.27)) hide)
     )
+    (pin "1")
   )
   (symbol (lib_id "power:GND") (at 194.31 76.2 0) (unit 1)
@@
       (effects (font (size 1.27 1.27)) hide)
     )
+    (pin "1")
   )
   (symbol (lib_id "power:Earth") (at 238.76 91.44 0) (unit 1)
@@
       (effects (font (size 1.27 1.27)) hide)
     )
+    (pin "1")
   )
   (symbol (lib_id "Device:R_Small") (at 184.15 83.82 90) (unit 1)
@@
       (effects (font (size 1.27 1.27)) hide)
     )
+    (pin "1")
+    (pin "2")
   )
   (symbol (lib_id "Device:R_Small") (at 199.39 35.56 90) (unit 1)
@@
       (effects (font (size 1.27 1.27)) hide)
     )
+    (pin "1")
+    (pin "2")
   )
   (symbol (lib_id "Device:C_Small") (at 199.39 45.72 270) (unit 1)
@@
       (effects (font (size 1.27 1.27)) hide)
     )
+    (pin "1")
+    (pin "2")
   )
   (symbol (lib_id "Device:C_Small") (at 199.39 55.88 270) (unit 1)
@@
       (effects (font (size 1.27 1.27)) hide)
     )
+    (pin "1")
+    (pin "2")
   )
   (symbol (lib_id "Device:C_Small") (at 199.39 66.04 270) (unit 1)
@@
       (effects (font (size 1.27 1.27)) hide)
     )
+    (pin "1")
+    (pin "2")
   )
   (symbol (lib_id "Device:C_Small") (at 199.39 76.2 270) (unit 1)
@@
       (effects (font (size 1.27 1.27)) hide)
     )
+    (pin "1")
+    (pin "2")
   )
   (symbol (lib_id "local:KSZ9477S") (at 137.16 60.96 0) (unit 6)
     (in_bom yes) (on_board yes)
-    (property "Reference" "U1" (id 0) (at 139.7 40.64 0))
+    (property "Reference" "U" (id 0) (at 139.7 40.64 0))
     (property "Value" "KSZ9477S" (id 1) (at 139.7 43.18 0))
     (property "Footprint" "footprints:TQFP-128_14x14mm_P0.4mm_EP10x10mm_ThermalVias" (id 2) (at 121.666 82.042 0)
@@
       (effects (font (size 1.27 1.27)) hide)
     )
+    (pin "115")
+    (pin "116")
+    (pin "117")
+    (pin "118")
+    (pin "120")
+    (pin "112")
+    (pin "113")
+    (pin "121")
+    (pin "102")
+    (pin "103")
   )
   (symbol (lib_id "Connector:JK0654219") (at 238.76 60.96 0) (unit 1)
@@
       (effects (font (size 1.27 1.27)) hide)
     )
+    (pin "1")
+    (pin "10")
+    (pin "11")
+    (pin "12")
+    (pin "13")
+    (pin "14")
+    (pin "15")
+    (pin "16")
+    (pin "2")
+    (pin "3")
+    (pin "4")
+    (pin "5")
+    (pin "6")
+    (pin "7")
+    (pin "8")
+    (pin "9")
+    (pin "SH")
   )
   (sheet (at 38.1 25.4) (size 64.77 50.8)
@@
       (effects (font (size 1.27 1.27)) (justify left bottom))
     )
-    (property "Sheet file" "ethernet_ports_1_2.kicad_sch" (id 1) (at 38.1 76.7089 0)
+    (property "Dateiname Blatt" "ethernet_ports_1_2.kicad_sch" (id 1) (at 38.1 76.7089 0)
       (effects (font (size 1.27 1.27)) (justify left top))
     )
@@
       (effects (font (size 1.27 1.27)) (justify left bottom))
     )
-    (property "Sheet file" "ethernet_ports_3_4.kicad_sch" (id 1) (at 38.1 140.2089 0)
+    (property "Dateiname Blatt" "ethernet_ports_3_4.kicad_sch" (id 1) (at 38.1 140.2089 0)
       (effects (font (size 1.27 1.27)) (justify left top))
     )
